File: hardware/riv_cosmici.kicad_pcb (KiCad board)
At the start: 2 copper layers, 80 x 55 mm, 59 parts, among them J1 SiPM, J2 TTL_OUT, J3 PWR_5V, Q1 BFR93A, Q2 MMBTH81, U1 LT3461, U2 TLC555/LMC555, U3 MAX961, U4 MCP1402, U5 LP2985AIM5-3.6, U6 MCP1825S-3302, U7 LP2985AIM5-3.6, U8 LT1636

Commit message: Scheda completa: simulazione LTspice, correzione V2, uscita 3,3 V per Raspberry Pi
- Schema KiCad confrontato pin per pin con l'originale INFN: V2 e' un
  potenziometro (cursore -> R17 -> TH), non un reostato. Corretto.
- Uscita J4 per Raspberry Pi: il buffer a 2 transistor a 5 V (lento,
  uscita fino a -0,7 V, 5 V sui GPIO) sostituito da U9 74LVC1G17 a +3V3
  + R23 33 ohm. Buffer ora anche su PCB e Gerber.
- PCB rigenerato (autorouter con rip-up & retry): 0 errori DRC e
  connettivita'. Gerber + zip, anteprime, riv.kicad_sym, BOM generata
  da netdata.py (gen_bom.py).
- simulation/ltspice/: scheda intera come schema LTspice (.asc + .asy)
  e netlist (.cir), generati dallo stesso modello dati del KiCad;
  macromodelli di tutti gli integrati; verifica_ltspice.py controlla
  .asc == .cir e 21 grandezze con ngspice (tutte OK).
- netlist_from_kicad: PWR_FLAG non e' piu' trattato come una rete.
- hardware/PRIMA_DI_ORDINARE.md: verifiche fatte e punti da decidere
  al montaggio (R3/limite 40 V LT3461, condensatori LDO, L1, LEMO).

Co-Authored-By: Claude Opus 5.5 <noreply@anthropic.com>
Claude-Session: https://claude.ai/code/session_017fc9yPsNewCQrMK8R1c8Ls
Parts:
- added CF10: 100n, rivlib:C_0805, F.Cu at (88.0, 48.5)
- added J4: LEMO_OUT, rivlib:HDR1x02, F.Cu at (97.0, 54.0)
- added R23: 33R, rivlib:R_0805, F.Cu at (92.5, 52.5)
- added U9: 74LVC1G17, rivlib:SOT23-5, F.Cu at (88.0, 52.5)
Connections:
- R19 pad 1: TH_W -> TH_HI
- V2 pad 1: TH_W -> TH_HI
Routing:
- net CMP_Q: track 22.2 -> 63.1 mm, vias 2 -> 4
- net +3V3: track 104.0 -> 123.3 mm
- net TH_HI: track 0.00 -> 14.1 mm
- net CMP_QB: track 25.5 -> 18.1 mm, vias 2 -> 0
- net CTL555: track 30.9 -> 26.5 mm
- net GND: track 68.9 -> 73.2 mm, vias 40 -> 42
- net BUF_Y: track 0.00 -> 4.23 mm
- net TH_LO: track 14.9 -> 11.6 mm, vias 0 -> 1
- net TH_W: track 12.5 -> 9.76 mm
- net T555: track 25.5 -> 28.2 mm
- net BUF_OUT: track 0.00 -> 2.39 mm
- net LED_K: track 6.56 -> 7.22 mm

Commit message: Verifica con KiCad 7: corretti collegamenti ai pad, isole di massa e giunzioni dello schema
Il DRC di KiCad ha trovato reti aperte che il controllo interno non vedeva:
- piste che toccavano solo l'angolo del rettangolo d'ingombro di pad tondi o
  arrotondati: ora ogni pista viene prolungata fino al centro del pad
  (gen_pcb.snap_to_pads) e la connettivita' si controlla sulla forma reale;
  pad SMD rettangolari anche in KiCad, come nei Gerber;
- isole del piano di massa staccate (prima i pezzi del piano contavano come uno):
  niente colli sotto 0,3 mm, reti che chiudono le isole ri-instradate per prime,
  pista di massa aggiunta sulla scheda a 3 canali; scheda a 1 canale ri-instradata;
- giunzioni a T nello schema (Q1C, LE) non collegate da KiCad: fili spezzati in
  ogni giunzione.

Nuovo generator/verifica_kicad.py: netlist dello schema (kicad-cli) = PCB, DRC di
KiCad, connettivita' sul rame reale. Entrambe le schede: OK.
Gerber, JLCPCB, zip KiCad, PDF e render rigenerati.

Co-Authored-By: Claude Opus 5.5 <noreply@anthropic.com>
Claude-Session: https://claude.ai/code/session_017fc9yPsNewCQrMK8R1c8Ls
Routing:
- net +5V: track 189.0 -> 212.0 mm, vias 5 -> 6
- net +3V3: track 123.3 -> 136.8 mm, vias 6 -> 2
- net CMP_Q: track 63.1 -> 52.9 mm, vias 4 -> 3
- net CTL555: track 26.5 -> 16.6 mm
- net Q1C: track 16.5 -> 21.5 mm, vias 0 -> 2
- net VOUT40: track 48.6 -> 52.9 mm
- net FB: track 27.4 -> 30.7 mm
- net SW: track 5.34 -> 8.29 mm
- net GND: track 73.2 -> 75.8 mm
- net Q1B: track 17.8 -> 20.3 mm, vias 0 -> 2
- net SIG_IN: track 20.3 -> 22.8 mm
- net T555: track 28.2 -> 30.6 mm
- net VREF_B: track 13.3 -> 15.6 mm
- net TH_LO: track 11.6 -> 13.8 mm
- net LE: track 10.2 -> 12.3 mm
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
Commit message: KiCad 10: nomi delle reti del PCB allineati allo schema, VOUT del LT3461 come uscita di alimentazione
- allinea_reti_kicad.py (chiamato da gen_variante3): le reti del PCB prendono i nomi
  che KiCad ricava dallo schema (/ETICHETTA, Net-(...), unconnected-(...)), dopo aver
  verificato che i collegamenti coincidono: elimina i 199 net_conflict del DRC con
  --schematic-parity.
- LT3461 pin 5 (CAP/VOUT) di tipo power_out: risolve l'unico power_pin_not_driven
  dell'ERC (VOUT40 alimenta i V+ dei tre LT1636).
Verifica KiCad su entrambe le schede: OK.

Co-Authored-By: Claude Opus 5.5 <noreply@anthropic.com>
Claude-Session: https://claude.ai/code/session_017fc9yPsNewCQrMK8R1c8Ls
Connections:
- net BIAS renamed /BIAS
- net BUF_OUT renamed Net-(J4-Pad1)
- net BUF_Y renamed Net-(U9-Y)
- net CMP_IN renamed /CMP_IN
- net CMP_Q renamed /CMP_Q
- net CMP_QB renamed /CMP_QB
- net CTL555 renamed Net-(U2-CTL)
- net FB renamed Net-(U1-FB)
- net INV renamed Net-(U8--)
- net LE renamed Net-(U3-LE)
- net LED_A renamed Net-(U2-Q)
- net LED_K renamed Net-(D3-A)
- net Q1B renamed Net-(Q1-B)
- net Q1C renamed Net-(Q1-C)
- net Q2C renamed Net-(Q2-C)
- net Q2E renamed Net-(Q2-E)
- net SIG_IN renamed Net-(C7-Pad1)
- net SW renamed Net-(U1-SW)
- net T555 renamed Net-(U2-DIS)
- net TH renamed /TH
- net TH_HI renamed Net-(R19-Pad1)
- net TH_LO renamed Net-(R18-Pad1)
- net TH_W renamed Net-(V2-W)
- net TTL_OUT renamed Net-(U4-OUT)
- net VADJ_HI renamed Net-(D1-K)
- net VADJ_LO renamed Net-(R7-Pad1)
- net VOUT40 renamed /VOUT40
- net VREF_B renamed Net-(D1-A)
- net VREG38 renamed Net-(R5-Pad2)
- net VSET renamed Net-(U8-+)
- U5 pad 4: (no net) -> unconnected-(U5-BYP-Pad4)
- U7 pad 4: (no net) -> unconnected-(U7-BYP-Pad4)
- U8 pad 1: (no net) -> unconnected-(U8-NC-Pad1)
- U8 pad 5: (no net) -> unconnected-(U8-NC-Pad5)
- U8 pad 8: (no net) -> unconnected-(U8-NC-Pad8)
- U9 pad 1: (no net) -> unconnected-(U9-NC-Pad1)

Commit message: R3 = 255k e 2,2 uF su CF4/CF7/CF9 (datasheet LT3461, LP2985, MCP1825), nota per la verifica INFN
- R3 270k -> 255k: VOUT40 da 41,7 a 39,4 V, sotto i 40 V max assoluti del LT3461;
  bias ancora regolabile fino a ~39,2 V (margine 1,0 V a 25 C, 0,3 V a 50 C).
- CF4, CF7, CF9 100n -> 2,2 uF X7R 0805 (Samsung CL21B225KAFNNNE): uscite dei
  regolatori, come richiesto dai datasheet.
- Schemi, PCB (valori), BOM, file JLCPCB, PDF, simulazioni e render rigenerati;
  verifica_ltspice: tutto OK; sim_3canali invariata salvo VOUT40.
- hardware/variante_3ch/NOTA_PER_TECNICO_INFN.txt: le due modifiche con calcoli,
  simulazioni e punti da verificare, piu' l'elenco delle differenze dalla scheda INFN.

Co-Authored-By: Claude Opus 5.5 <noreply@anthropic.com>
Claude-Session: https://claude.ai/code/session_017fc9yPsNewCQrMK8R1c8Ls
Parts:
- CF4, CF7, CF9: value 100n -> 2.2uF
- R3: value 270k -> 255k
