File: hardware/variante_3ch/riv_cosmici_3ch.kicad_sch (KiCad schematic)
At the start: 203 parts, among them J101 SiPM_CH1, J104 LEMO_CH1, J201 SiPM_CH2, J204 LEMO_CH2, J3 PWR_5V, J301 SiPM_CH3, J304 LEMO_CH3, J5 LEMO_AND, J6 I2C_RPI, Q101 BFR93A, Q102 MMBTH81, Q201 BFR93A, Q202 MMBTH81, Q301 BFR93A, Q302 MMBTH81, U1 LT3461, U10 74LVC1G11, U102 TLC555/LMC555, U103 MAX961, U108 LT1636, U109 74LVC1G17, U11 MCP3424, U202 TLC555/LMC555, U203 MAX961, U208 LT1636, U209 74LVC1G17, U302 TLC555/LMC555, U303 MAX961, U308 LT1636, U309 74LVC1G17, U5 LP2985AIM5-3.6, U6 MCP1825S-3302, U7 LP2985AIM5-3.6

Commit message: Monitor: J6 Molex KK 254 a 3 poli (22-27-2031) come i connettori delle barre
Footprint MOLEX_KK_3, J6 spostato in orizzontale nel blocco MONITOR (il corpo del KK
sporgeva dal bordo); ri-instradate solo I2C_SDA e I2C_SCL (reinstrada_reti3.py),
resto del routing invariato. DRC 0, connettivita' OK, verifica KiCad OK.
Lista Mouser: 22-27-2031 x3, 22-01-3037 x3, contatti 08-50-0114 x30.
Serigrafia, Gerber, JLCPCB, PDF, zip KiCad, modello 3D e render aggiornati.

Co-Authored-By: Claude Opus 5.5 <noreply@anthropic.com>
Claude-Session: https://claude.ai/code/session_017fc9yPsNewCQrMK8R1c8Ls
Parts:
- J6: footprint rivlib:HDR1x03 -> rivlib:MOLEX_KK_3

Commit message: Secondo ADC per soglie e temperatura: PCB a 3 canali rifatto e verificato (103 x 223,9 mm)
- routing completo con il nuovo blocco MONITOR (U11 + U12 affiancati, termistore, J6)
  e la lettura delle soglie (R?52 10k + C?52 100n accanto al pin 2 del comparatore):
  0 reti fallite, DRC 0, connettivita' OK; verifica KiCad: schema = PCB, nessun errore,
  0 reti spezzate sul rame reale.
- regola di distanza piste del monitor <-> nodi sensibili resa simmetrica (1,2 mm su
  entrambi gli strati): rifatte Q1B3, Q2C2, MON3 (MON3 fuori dalla zona dell'uscita
  del canale 2, niente isole di massa), CMP_IN2 e MONTH2; ingresso comparatore
  20,6-20,9 mm in tutti e tre i canali, senza vie.
- C11 spostato di 1,27 mm (spazio per le scritte di C52/R52); serigrafia 0805 con i
  trattini tra i pad (niente contorni che si toccano: silk_overlap 0).
- Gerber, JLCPCB (U11+U12 MCP3424, RT1 NCP21XV103J03RA, R44 22k), stampa 1:1, schemi,
  zip KiCad, render rigenerati; tolto l'avviso 'lavoro in corso'.

Co-Authored-By: Claude Opus 5.5 <noreply@anthropic.com>
Claude-Session: https://claude.ai/code/session_017fc9yPsNewCQrMK8R1c8Ls
Parts:
- added C152, C252, C352, C41, CF13: 100n, rivlib:C_0805, symbol riv:C
- added R152, R252, R352: 10k, rivlib:R_0805, symbol riv:R
- added R44: 22k, rivlib:R_0805, symbol riv:R
- added RT1: 10k NTC, rivlib:R_0805, symbol riv:R
- added U12: MCP3424, rivlib:SOIC14, symbol riv:MCP3424
Connections:
- net +3V3: now also CF13.1, R44.1, U12.6 (VDD), U12.9 (A0)
- net GND: now also C152.2, C252.2, C352.2, C41.2, CF13.2, RT1.2, U12.10 (A1), U12.12 (CH3-), U12.14 (CH4-), U12.2 (CH1-), U12.4 (CH2-), U12.5 (VSS)
- net SCL_ADC: now also U12.8 (SCL)
- net SDA_ADC: now also U12.7 (SDA)
- net TH1: now also R152.1
- net TH2: now also R252.1
- net TH3: now also R352.1
- new net MONT: C41.1, R44.2, RT1.1, U12.13 (CH4+)
- new net MONTH1: C152.1, R152.2, U12.1 (CH1+)
- new net MONTH2: C252.1, R252.2, U12.3 (CH2+)
- new net MONTH3: C352.1, R352.2, U12.11 (CH3+)
Other:
- note added: "Adr0 = VDD, Adr1 = GND: indirizzo diverso da U11"
- note added: "MONITOR SOGLIE E TEMPERATURA: TH -> 10k + 100n (accanto al comparatore) -> ADC MCP3424 U12 (I2C)"
- note added: "NTC 10k: temperatura"
- note added: "PARTI COMUNI: boost 39,4 V, 3,3 V, riferimenti 3,6 V"
- note removed: "PARTI COMUNI: boost 41,7 V, 3,3 V, riferimenti 3,6 V"
- moved on the sheet: MH1, MH2, MH3, MH4, MH5, MH6, MH7, MH8

Commit message: Scheda a 3 canali: protezione dell'alimentazione (USB-C, fusibile, TVS, MOSFET P, LED)
USB-C solo alimentazione J7 (GCT USB4125-GF-A, 5,1k su CC) o J3 da banco ->
fusibile ripristinabile F1 (MF-MSMF050-2) -> TVS D5 (SMAJ5.0A) -> MOSFET P Q4
(AO3401A, inversione di polarita') -> +5V; C60 10 uF e LED di accensione D6.
Generatore: piazzole con asola (guscio USB-C) in PCB KiCad, Gerber e foratura (G85);
nuovi simboli e impronte (dalla libreria KiCad 7.0.11); routing aggiunto senza toccare
le altre reti. Verifica KiCad: schema = PCB, DRC senza errori, 0 reti spezzate.
Simulazione ngspice della scheda intera: +5V 4,977 V, il resto invariato.
Schema A4: nuovo foglio 2 (ingresso e protezione); nota per il tecnico INFN aggiornata.

Co-Authored-By: Claude Opus 5.5 <noreply@anthropic.com>
Claude-Session: https://claude.ai/code/session_017fc9yPsNewCQrMK8R1c8Ls
Parts:
- added C60: 10u, rivlib:C_1206, symbol riv:C
- added D5: SMAJ5.0A, rivlib:D_SMA, symbol riv:TVS
- added D6: LED verde, rivlib:LED_0805, symbol riv:LED
- added F1: MF-MSMF050-2, rivlib:F_1812, symbol riv:FUSE
- added J7: USB_C_PWR, rivlib:USBC_GCT_USB4125, symbol riv:USBC
- added Q4: AO3401A, rivlib:SOT23, symbol riv:PMOS
- added R60, R61: 5k1, rivlib:R_0805, symbol riv:R
- added R62: 10k, rivlib:R_0805, symbol riv:R
- added R63: 1k5, rivlib:R_0805, symbol riv:R
Connections:
- net +5V: now also C60.1, Q4.2 (S), R63.1; no longer J3.2
- net GND: now also C60.2, D5.2 (A), D6.1 (K), J7.4 (GND), R60.2, R61.2, R62.2
- new net CC1: J7.2 (CC1), R60.1
- new net CC2: J7.3 (CC2), R61.1
- new net LED_PWR: D6.2 (A), R63.2
- new net Q4_G: Q4.1 (G), R62.1
- new net VIN_F: D5.1 (K), F1.2, Q4.3 (D)
- new net VIN_RAW: F1.1, J3.2, J7.1 (VBUS)
Other:
- note added: "5,1k: il caricatore da' 5 V"
- note added: "LED acceso"
- note added: "MONITOR TENSIONI: partitori 1M/43k su VREG38n e VOUT40 -> ADC MCP3424 (I2C, 0x68) -> J6"
- note added: "PROTEZIONE ALIMENTAZIONE: USB-C o J3 -> fusibile F1 -> TVS D5 -> MOSFET P Q4 (inversione) -> +5V"
- note added: "SOLO 5 V (banco)"
- note added: "USB-C solo alimentazione"
- note added: "verso la scatolina di acquisizione (pull-up li')"
- note removed: "+5V IN"
- note removed: "MONITOR TENSIONI: partitori 1M/43k su VREG38n e VOUT40 -> ADC MCP3424 (I2C, 0x68) -> Raspberry Pi"
- note removed: "verso Raspberry Pi (pull-up sul Pi)"
